File: PLC homemade/Ethernet.kicad_sch (KiCad schematic)
At the start: 0 parts

Commit message: :chart_with_upwards_trend:COMPLETED EHERNET, left 1 component out
Parts:
- added C10, C11, C12, C13, C14, C9: 100nF 50V, symbol Device:C
- added C15, C16: 20pF, symbol Device:C
- added C17: 22nF, symbol Device:C
- added C18, C8: 10nF 25V, symbol Device:C
- added C19: 6.8nF, symbol Device:C
- added C20: 82R, symbol Device:C
- added C7: 4.7uF 6.3V, symbol Device:C
- added R10, R11, R12, R16, R21, R4, R5, R6, R7, R8, R9: 10K, symbol Device:R
- added R13: 12.4K/1%, symbol Device:R
- added R14: RC0402FR-070RL, symbol Device:R
- added R15: 1M, symbol Device:R
- added R17, R18: 49.9R, symbol Device:R
- added R19, R20: 510R, symbol Device:R
- added R22: 82R, symbol Device:R
- added U3: W5500, Package_QFP:LQFP-48_7x7mm_P0.5mm, symbol Interface_Ethernet:W5500
- added Y1: Crystal, symbol Device:Crystal
Connections:
- new net: R13.1, U3.10 (EXRES1)
- new net: C7.1, U3.20 (TOCAP)
- new net: C8.1, U3.22 (1V2O)
- new net: R12.2, U3.23 (RSVD)
- new net: R7.2, U3.38 (RSVD)
- new net: R8.2, U3.39 (RSVD)
- new net: R9.2, U3.40 (RSVD)
- new net: R10.2, U3.41 (RSVD)
- new net: R11.2, U3.42 (RSVD)
- new net: R6.2, U3.43 (PMODE2)
- new net: R5.2, U3.44 (PMODE1)
- new net: R4.2, U3.45 (PMODE0)
- new net 3V3: R14.1
- new net 3V3NET: C10.1, C11.1, C12.1, C13.1, C14.1, C9.1, R14.2, R16.2, R17.2, R18.2, R4.1, R5.1, R6.1, U3.11 (AVDD), U3.15 (AVDD), U3.17 (AVDD), U3.21 (AVDD), U3.28 (VDD), U3.4 (AVDD), U3.8 (AVDD)
- new net ACT: R19.2
- new net EMAC_CLK: U3.33 (SCLK)
- new net EMAC_CS: U3.32 (~{SCS})
- new net EMAC_INT: U3.36 (~{INT})
- new net EMAC_MISO: U3.34 (MISO)
- new net EMAC_MOSI: U3.35 (MOSI)
- new net EMAC_RST: U3.37 (~{RST})
- new net GND: C10.2, C11.2, C12.2, C13.2, C14.2, C15.2, C16.2, C17.2, C18.1, C7.2, C8.2, C9.2, R10.1, R11.1, R12.1, R13.2, R15.1, R7.1, R8.1, R9.1, U3.14 (AGND), U3.16 (AGND), U3.19 (AGND), U3.29 (GND), U3.3 (AGND), U3.48 (AGND), U3.9 (AGND)
- new net LED_ACT: U3.27 (ACTLED)
- new net LED_LINK: U3.25 (LINKLED)
- new net LINK: R20.2
- new net PG: R15.2
- new net RCT: C18.2, R21.1, R22.1
- new net RXI_N: C20.1, C20.2, R22.2
- new net RXI_P: C19.1, C19.2, R21.2
- new net RX_N: U3.5 (RXN)
- new net RX_P: U3.6 (RXP)
- new net TCT: C17.1, R16.1
- new net TXI_N: R18.1
- new net TXI_P: R17.1
- new net TX_N: U3.1 (TXN)
- new net TX_P: U3.2 (TXP)
- new net XI: C15.1, U3.30 (XI/CLKIN), Y1.1
- new net XO: C16.1, U3.31 (XO), Y1.2
- no-connect marks 0 -> 3
Other:
- added sheet Sheet03 (Sheet03.kicad_sch)

Commit message: :green_heart: CoRRECTED pOWER eRRORS
Connections:
- net LED_ACT: now also R19.1
- net LED_LINK: now also R20.1
- net 3V3 renamed 3.3V

Commit message: :art: COMPLETED SHEET3
Parts:
- added J7: SS-74810-004, SS-74810-004:BEL_SS-74810-004, symbol SS-74810-004:SS-74810-004
Connections:
- net 3V3NET: now also J7.11_1, J7.11_2, J7.9_1, J7.9_2
- net ACT: now also J7.10_1, J7.10_2
- net GND: now also J7.S1 (SHIELD), J7.S2 (SHIELD), J7.S3 (SHIELD), J7.S4 (SHIELD), J7.S5 (SHIELD), J7.S6 (SHIELD), J7.S7 (SHIELD), J7.S8 (SHIELD), J7.S9 (SHIELD)
- net LINK: now also J7.12_1, J7.12_2
- net MH1: now also J7.4_2 (P4_2)
- net MH2: now also J7.8_2 (P8_2)
- net RCT: now also J7.5_1 (P5_1), J7.5_2 (P5_2)
- net RXI_P: now also J7.6_1 (P6_1), J7.6_2 (P6_2), J7.7_1 (P7_1), J7.7_2 (P7_2)
- net TCT: now also J7.3_1 (P3_1), J7.3_2 (P3_2)
- net TXI_N: now also J7.2_1 (P2_1), J7.2_2 (P2_2)
- net TXI_P: now also J7.1_1 (P1_1), J7.1_2 (P1_2)
- no-connect marks 3 -> 5
Other:
- note added: "ETHERNET"
- moved on the sheet: C10, C11, C12, C13, C14, C15, C16, C17, C18, C19, C20, C7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

Commit message: :clown_face: changed HEIRACHIAL to global
Parts:
- removed unit 2 of J7
Connections:
- net MH1: now also J7.4_1 (P4_1)
- net MH2: now also J7.8_1 (P8_1)
- no-connect marks 5 -> 3
Other:
- moved on the sheet: J7A

Commit message: :tada: Added small changes
Changed lines of the file:
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@@
 		)
 	)
-	(hierarchical_label "EMAC_INT"
+	(global_label "EMAC_RST"
 		(shape input)
-		(at 46.99 64.77 180)
+		(at 46.99 67.31 180)
+		(fields_autoplaced yes)
 		(effects
 			(font
@@
 			(justify right)
 		)
+		(property "Intersheetrefs" "${INTERSHEET_REFS}"
+			(at 34.6311 67.31 0)
+			(effects
+				(font
+					(size 1.27 1.27)
+				)
+				(justify right)
+				(hide yes)
+			)
+		)
 	)
-	(hierarchical_label "EMAC_MOSI"
+	(global_label "EMAC_INT"
 		(shape input)
-		(at 46.99 62.23 180)
+		(at 46.99 64.77 180)
+		(fields_autoplaced yes)
 		(effects
 			(font
@@
 			(justify right)
 		)
+		(property "Intersheetrefs" "${INTERSHEET_REFS}"
+			(at 35.1753 64.77 0)
+			(effects
+				(font
+					(size 1.27 1.27)
+				)
+				(justify right)
+				(hide yes)
+			)
+		)
 	)
-	(hierarchical_label "EMAC_MISO"
+	(global_label "EMAC_MOSI"
 		(shape input)
-		(at 46.99 59.69 180)
+		(at 46.99 62.23 180)
+		(fields_autoplaced yes)
 		(effects
 			(font
@@
 			(justify right)
 		)
+		(property "Intersheetrefs" "${INTERSHEET_REFS}"
+			(at 33.482 62.23 0)
+			(effects
+				(font
+					(size 1.27 1.27)
+				)
+				(justify right)
+				(hide yes)
+			)
+		)
 	)
-	(hierarchical_label "EMAC_CLK"
+	(global_label "EMAC_MISO"
 		(shape input)
-		(at 46.99 57.15 180)
+		(at 46.99 59.69 180)
+		(fields_autoplaced yes)
 		(effects
 			(font
@@
 			(justify right)
 		)
+		(property "Intersheetrefs" "${INTERSHEET_REFS}"
+			(at 33.482 59.69 0)
+			(effects
+				(font
+					(size 1.27 1.27)
+				)
+				(justify right)
+				(hide yes)
+			)
+		)
 	)
-	(hierarchical_label "EMAC_CS"
+	(global_label "EMAC_CLK"
 		(shape input)
-		(at 46.99 54.61 180)
+		(at 46.99 57.15 180)
+		(fields_autoplaced yes)
 		(effects
 			(font
@@
 			(justify right)
 		)
+		(property "Intersheetrefs" "${INTERSHEET_REFS}"
+			(at 34.5101 57.15 0)
+			(effects
+				(font
+					(size 1.27 1.27)
+				)
+				(justify right)
+				(hide yes)
+			)
+		)
 	)
-	(hierarchical_label "EMAC_RST"
+	(global_label "EMAC_CS"
 		(shape input)
-		(at 46.99 67.31 180)
+		(at 46.99 54.61 180)
+		(fields_autoplaced yes)
 		(effects
 			(font
@@
 			(justify right)
 		)
+		(property "Intersheetrefs" "${INTERSHEET_REFS}"
+			(at 35.5987 54.61 0)
+			(effects
+				(font
+					(size 1.27 1.27)
+				)
+				(justify right)
+				(hide yes)
+			)
+		)
 	)

Commit message: :tada: Run Electrical rule checker All errors corrected
Parts:
- C10, C11, C12, C13, C14, C15, C16, C17, C18, C19, C7, C8, C9: footprint (none) -> Capacitor_SMD:C_01005_0402Metric
- C20: value 82R -> 6.8nF; footprint (none) -> Capacitor_SMD:C_01005_0402Metric
- R10, R11, R12, R13, R14, R15, R16, R21, R4, R5, R6, R7, R8, R9: footprint (none) -> Resistor_SMD:R_01005_0402Metric
- R17, R18, R19, R20, R22: footprint (none) -> Resistor_SMD:R_1206_3216Metric
- Y1: footprint (none) -> Crystal:Crystal_SMD_5032-2Pin_5.0x3.2mm
Connections:
- net MH1 is gone; now on net GND: J7.4_1 (P4_1)
- net MH2 is gone; now on net GND: J7.8_1 (P8_1)
- net TX_N is gone; now on net TXI_N: U3.1 (TXN)
- net TX_P is gone; now on net TXI_P: U3.2 (TXP)
- net RXI_N: now also J7.7_1 (P7_1); no longer C20.1, R22.2
- net RXI_P: no longer C19.1, J7.7_1 (P7_1), R21.2
- net RX_N: now also C20.1, R22.2
- net RX_P: now also C19.1, R21.2
