File: PLC homemade/Sheet04.kicad_sch (KiCad schematic)
At the start: 0 parts

Commit message: :spanner:At interfaces
Parts:
- added C29: 100nF 50V, symbol Device:C
- added R36, R37, R38, R39, R40, R41: 4K7, symbol Device:R
Connections:
- new net 3V3: C29.1
- new net GND: C29.2

Commit message: :rocket: started on OUTPUT
Parts:
- added IC1: PCF8574DGVR, PCF8574DGVR:DIL16, symbol PCF8574DGVR:PCF8574DGVR
- added J2: 1803316, 1803316:PHOENIX_1803316, symbol 1803316:1803316
Connections:
- net 3V3: now also R36.2, R37.2, R38.2, R39.2, R40.2, R41.2, IC1.16 (VCC), IC1.3 (A2)
- net GND: now also IC1.1 (A0), IC1.2 (A1), IC1.8 (GND)
- net INPUT_D1: now also J2.01
- net INPUT_D2: now also J2.02
- net INPUT_D3: now also J2.03
- net INPUT_D4: now also J2.04
- net INPUT_D5: now also J2.05
- net INPUT_D6: now also J2.06
- net IN_D1: now also R36.1, IC1.4 (P0)
- net IN_D2: now also R37.1, IC1.5 (P1)
- net IN_D3: now also R38.1, IC1.6 (P2)
- net IN_D4: now also R39.1, IC1.7 (P3)
- net IN_D5: now also R40.1, IC1.9 (P4)
- net IN_D6: now also R41.1, IC1.10 (P5)
- new net IIC_SCL: IC1.14 (SCL)
- new net IIC_SDA: IC1.15 (SDA)
- no-connect marks 0 -> 3
Other:
- added sheet OUTPUT (OUTPUT.kicad_sch)

Commit message: :green_heart: CoRRECTED pOWER eRRORS
Connections:
- net 3V3 renamed 3.3V
Changed lines of the file:
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@@
 	(wire
 		(pts
-			(xy 179.07 22.86) (xy 179.07 16.51)
+			(xy 179.07 22.86) (xy 179.07 19.05)
 		)
 		(stroke
@@
 		)
 	)
+	(label "IN_D4"
+		(at 125.73 81.28 0)
+		(effects
+			(font
+				(size 1.27 1.27)
+			)
+			(justify left bottom)
+		)
+	)
+	(label "IN_D3"
+		(at 125.73 73.66 0)
+		(effects
+			(font
+				(size 1.27 1.27)
+			)
+			(justify left bottom)
+		)
+	)
+	(label "IN_D2"
+		(at 125.73 67.31 0)
+		(effects
+			(font
+				(size 1.27 1.27)
+			)
+			(justify left bottom)
+		)
+	)
+	(label "IN_D1"
+		(at 125.73 60.96 0)
+		(effects
+			(font
+				(size 1.27 1.27)
+			)
+			(justify left bottom)
+		)
+	)
 	(label "IN_D5"
 		(at 125.73 87.63 0)
@@
 	)
 	(label "IN_D4"
-		(at 125.73 81.28 0)
-		(effects
-			(font
-				(size 1.27 1.27)
-			)
-			(justify left bottom)
-		)
-	)
-	(label "IN_D2"
-		(at 125.73 67.31 0)
-		(effects
-			(font
-				(size 1.27 1.27)
-			)
-			(justify left bottom)
-		)
-	)
-	(label "IN_D3"
-		(at 125.73 73.66 0)
-		(effects
-			(font
-				(size 1.27 1.27)
-			)
-			(justify left bottom)
-		)
-	)
-	(label "IN_D1"
-		(at 125.73 60.96 0)
-		(effects
-			(font
-				(size 1.27 1.27)
-			)
-			(justify left bottom)
-		)
-	)
-	(label "IN_D4"
 		(at 227.33 57.15 180)
 		(effects
@@
 			)
 			(justify right bottom)
-		)
-	)
-	(label "3V3"
-		(at 148.59 54.61 0)
-		(effects
-			(font
-				(size 1.27 1.27)
-			)
-			(justify left bottom)
-		)
-	)
-	(label "3V3"
-		(at 179.07 16.51 0)
-		(effects
-			(font
-				(size 1.27 1.27)
-			)
-			(justify left bottom)
-		)
-	)
-	(label "3V3"
-		(at 175.26 50.8 0)
-		(effects
-			(font
-				(size 1.27 1.27)
-			)
-			(justify left bottom)
 		)
 	)
@@
 	)
 	(symbol
+		(lib_id "power:+3.3V")
+		(at 148.59 54.61 0)
+		(unit 1)
+		(exclude_from_sim no)
+		(in_bom yes)
+		(on_board yes)
+		(dnp no)
+		(fields_autoplaced yes)
+		(property "Reference" "#PWR066"
+			(at 148.59 58.42 0)
+			(effects
+				(font
+					(size 1.27 1.27)
+				)
+				(hide yes)
+			)
+		)
+		(property "Value" "3.3V"
+			(at 148.59 49.53 0)
+			(effects
+				(font
+					(size 1.27 1.27)
+				)
+			)
+		)
+		(property "Footprint" ""
+			(at 148.59 54.61 0)
+			(effects
+				(font
+					(size 1.27 1.27)
+				)
+				(hide yes)
+			)
+		)
+		(property "Datasheet" ""
+			(at 148.59 54.61 0)
+			(effects
+				(font
+					(size 1.27 1.27)
+				)
+				(hide yes)
+			)
+		)
+		(property "Description" "Power symbol creates a global label with name \"+3.3V\""
+			(at 148.59 54.61 0)
+			(effects
+				(font
+					(size 1.27 1.27)
+				)
+				(hide yes)
+			)
+		)
+		(pin "1"
+		)
+		(instances
+			(project "PLC homemade"
+				(path "/152f83be-52d6-49bf-8437-949cb175c923/206ffe26-9c74-474c-9601-4af431c0356c/8fb64de6-c896-4577-8763-e28849f83596/6ac5e77b-6af3-438f-b539-14afc98dea7d"
+					(reference "#PWR066")
+					(unit 1)
+				)
+			)
+		)
+	)
+	(symbol
 		(lib_id "Device:R")
 		(at 139.7 81.28 90)
@@
 				(path "/152f83be-52d6-49bf-8437-949cb175c923/206ffe26-9c74-474c-9601-4af431c0356c/8fb64de6-c896-4577-8763-e28849f83596/6ac5e77b-6af3-438f-b539-14afc98dea7d"
 					(reference "R39")
+					(unit 1)
+				)
+			)
+		)
+	)
+	(symbol
+		(lib_id "power:+3.3V")
+		(at 179.07 19.05 0)
+		(unit 1)
+		(exclude_from_sim no)
+		(in_bom yes)
+		(on_board yes)
+		(dnp no)
+		(fields_autoplaced yes)
+		(property "Reference" "#PWR068"
+			(at 179.07 22.86 0)
+			(effects
+				(font
+					(size 1.27 1.27)
+				)
+				(hide yes)
+			)
+		)
+		(property "Value" "3.3V"
+			(at 179.07 13.97 0)
+			(effects
+				(font
+					(size 1.27 1.27)
+				)
+			)
+		)
+		(property "Footprint" ""
+			(at 179.07 19.05 0)
+			(effects
+				(font
+					(size 1.27 1.27)
+				)
+				(hide yes)
+			)
+		)
+		(property "Datasheet" ""
+			(at 179.07 19.05 0)
+			(effects
+				(font
+					(size 1.27 1.27)
+				)
+				(hide yes)
+			)
+		)
+		(property "Description" "Power symbol creates a global label with name \"+3.3V\""
+			(at 179.07 19.05 0)
+			(effects
+				(font
+					(size 1.27 1.27)
+				)
+				(hide yes)
+			)
+		)
+		(pin "1"
+		)
+		(instances
+			(project "PLC homemade"
+				(path "/152f83be-52d6-49bf-8437-949cb175c923/206ffe26-9c74-474c-9601-4af431c0356c/8fb64de6-c896-4577-8763-e28849f83596/6ac5e77b-6af3-438f-b539-14afc98dea7d"
+					(reference "#PWR068")
 					(unit 1)
 				)
@@
 					(unit 1)
 				)
+			)
+		)
+	)
+	(symbol
+		(lib_id "power:+3.3V")
+		(at 175.26 50.8 0)
+		(unit 1)
+		(exclude_from_sim no)
+		(in_bom yes)
+		(on_board yes)
+		(dnp no)
+		(fields_autoplaced yes)
+		(property "Reference" "#PWR067"
+			(at 175.26 54.61 0)
+			(effects
+				(font
+					(size 1.27 1.27)
+				)
+				(hide yes)
+			)
+		)
+		(property "Value" "3.3V"
+			(at 175.26 45.72 0)
+			(effects
+				(font
+					(size 1.27 1.27)
+				)
+			)
+		)
+		(property "Footprint" ""
+			(at 175.26 50.8 0)
+			(effects
+				(font
+					(size 1.27 1.27)
+				)
+				(hide yes)
+			)
+		)
+		(property "Datasheet" ""
+			(at 175.26 50.8 0)
+			(effects
+				(font
+					(size 1.27 1.27)
+				)
+				(hide yes)
+			)
+		)
+		(property "Description" "Power symbol creates a global label with name \"+3.3V\""
+			(at 175.26 50.8 0)
+			(effects
+				(font
+					(size 1.27 1.27)
+				)
+				(hide yes)
+			)
+		)
+		(pin "1"
+		)
+		(instances
+			(project "PLC homemade"
+				(path "/152f83be-52d6-49bf-8437-949cb175c923/206ffe26-9c74-474c-9601-4af431c0356c/8fb64de6-c896-4577-8763-e28849f83596/6ac5e77b-6af3-438f-b539-14afc98dea7d"
+					(reference "#PWR067")
+					(unit 1)
+				)

Commit message: :art: COMPLETED SHEET4
Parts:
- added R69, R70, R71, R72, R73, R74: 4K7 1206, symbol Device:R
- added U15, U16, U17, U18, U19, U20: EL357N-G, EL357N-G:OPTO_EL357N-G, symbol EL357N-G:EL357N-G
Connections:
- net GND: now also U15.3, U16.3, U17.3, U18.3, U19.3, U20.3
- net INPUT_D1: now also R69.1
- net INPUT_D2: now also R72.1
- net INPUT_D3: now also R70.1
- net INPUT_D4: now also R73.1
- net INPUT_D5: now also R71.1
- net INPUT_D6: now also R74.1
- net IN_D1: now also U15.4
- net IN_D2: now also U18.4
- net IN_D3: now also U16.4
- net IN_D4: now also U19.4
- net IN_D5: now also U17.4
- net IN_D6: now also U20.4
- new net: R70.2, U16.2
- new net: R71.2, U17.2
- new net: R73.2, U19.2
- new net: R72.2, U18.2
- new net: R69.2, U15.2
- new net: R74.2, U20.2
- new net +12V: U15.1, U16.1, U17.1, U18.1, U19.1, U20.1
Other:
- moved on the sheet: R36, R37, R38, R39, R40, R41

Commit message: :clown_face: changed HEIRACHIAL to global
Changed lines of the file:
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@@
 		)
 	)
-	(hierarchical_label "IIC_SCL"
+	(global_label "IIC_SDA"
 		(shape input)
-		(at 185.42 62.23 180)
+		(at 185.42 59.69 180)
+		(fields_autoplaced yes)
 		(effects
 			(font
@@
 			(justify right)
 		)
+		(property "Intersheetrefs" "${INTERSHEET_REFS}"
+			(at 175.4195 59.69 0)
+			(effects
+				(font
+					(size 1.27 1.27)
+				)
+				(justify right)
+				(hide yes)
+			)
+		)
 	)
-	(hierarchical_label "IIC_SDA"
+	(global_label "IIC_SCL"
 		(shape input)
-		(at 185.42 59.69 180)
+		(at 185.42 62.23 180)
+		(fields_autoplaced yes)
 		(effects
 			(font
@@
 			(justify right)
 		)
+		(property "Intersheetrefs" "${INTERSHEET_REFS}"
+			(at 175.48 62.23 0)
+			(effects
+				(font
+					(size 1.27 1.27)
+				)
+				(justify right)
+				(hide yes)
+			)
+		)
 	)

Commit message: :tada: Run Electrical rule checker All errors corrected
Parts:
- C29: footprint (none) -> Capacitor_SMD:C_01005_0402Metric
- R36, R37, R38, R39, R40, R41, R69, R70, R71, R72, R73, R74: footprint (none) -> Resistor_SMD:R_01005_0402Metric
Changed lines of the file:
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@@
 			)
 		)
-		(property "Footprint" ""
+		(property "Footprint" "Resistor_SMD:R_01005_0402Metric"
 			(at 153.67 72.898 90)
 			(effects
@@
 			)
 		)
-		(property "Footprint" ""
+		(property "Footprint" "Capacitor_SMD:C_01005_0402Metric"
 			(at 190.5 21.8948 0)
 			(effects
@@
 			)
 		)
-		(property "Footprint" ""
+		(property "Footprint" "Resistor_SMD:R_01005_0402Metric"
 			(at 153.67 86.868 90)
 			(effects
@@
 			)
 		)
-		(property "Footprint" ""
+		(property "Footprint" "Resistor_SMD:R_01005_0402Metric"
 			(at 29.21 55.118 90)
 			(effects
@@
 			)
 		)
-		(property "Footprint" ""
+		(property "Footprint" "Resistor_SMD:R_01005_0402Metric"
 			(at 153.67 80.518 90)
 			(effects
@@
 			)
 		)
-		(property "Footprint" ""
+		(property "Footprint" "Resistor_SMD:R_01005_0402Metric"
 			(at 153.67 66.548 90)
 			(effects
@@
 			)
 		)
-		(property "Footprint" ""
+		(property "Footprint" "Resistor_SMD:R_01005_0402Metric"
 			(at 85.09 34.798 90)
 			(effects
@@
 			)
 		)
-		(property "Footprint" ""
+		(property "Footprint" "Resistor_SMD:R_01005_0402Metric"
 			(at 153.67 60.198 90)
 			(effects
@@
 			)
 		)
-		(property "Footprint" ""
+		(property "Footprint" "Resistor_SMD:R_01005_0402Metric"
 			(at 30.48 30.988 90)
 			(effects
@@
 			)
 		)
-		(property "Footprint" ""
+		(property "Footprint" "Resistor_SMD:R_01005_0402Metric"
 			(at 83.82 57.658 90)
 			(effects
@@
 			)
 		)
-		(property "Footprint" ""
+		(property "Footprint" "Resistor_SMD:R_01005_0402Metric"
 			(at 85.09 79.248 90)
 			(effects
@@
 			)
 		)
-		(property "Footprint" ""
+		(property "Footprint" "Resistor_SMD:R_01005_0402Metric"
 			(at 153.67 93.218 90)
 			(effects
@@
 			)
 		)
-		(property "Footprint" ""
+		(property "Footprint" "Resistor_SMD:R_01005_0402Metric"
 			(at 30.48 75.438 90)
 			(effects
