File: PLC homemade/Sheet06.kicad_sch (KiCad schematic)
At the start: 9 parts, among them J5 USB4110GFA, U8 BC847BDW1T1G

Commit message: ::construction_worker:: Started on esp
Other:
- added sheet ESP (ESP.kicad_sch)
Changed lines of the file:
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@@
+		)
+	)
+	(sheet
+		(at 207.01 137.16)
+		(size 60.96 25.4)
+		(exclude_from_sim no)
+		(in_bom yes)
+		(on_board yes)
+		(dnp no)
+		(fields_autoplaced yes)
+		(stroke
+			(width 0.1524)
+			(type solid)
+		)
+		(fill
+			(color 0 0 0 0.0000)
+		)
+		(property "Sheetname" "ESP"
+			(at 207.01 136.4484 0)
+			(effects
+				(font
+					(size 1.27 1.27)
+				)
+				(justify left bottom)
+			)
+		)
+		(property "Sheetfile" "ESP.kicad_sch"
+			(at 207.01 163.1446 0)
+			(effects
+				(font
+					(size 1.27 1.27)
+				)
+				(justify left top)
+			)
+		)
+		(instances
+			(project "PLC homemade"
+				(path "/152f83be-52d6-49bf-8437-949cb175c923/206ffe26-9c74-474c-9601-4af431c0356c/8fb64de6-c896-4577-8763-e28849f83596/6ac5e77b-6af3-438f-b539-14afc98dea7d/58e05c6e-6b39-4026-a2a7-0a1b1e19bf35/65c884d1-f87c-4356-98e0-ebde83caffd4"
+					(page "7")
+				)
+			)
 		)
 	)

Commit message: :clown_face:Completed schematic
Parts:
- added C49, C50, C51: 100nF 50V, symbol Device:C
- added C52: 10uF 50V, symbol Device:C
- added Card1: TF PUSH, TF PUSH:TF-SMD_TF-PUSH, symbol TF PUSH:TFPUSH
- added D8: SLPRT5V0U2X, SLPRT5V0U2X:SOT-143-4_L2.9-W1.3-P1.90-LS2.4-BL, symbol SLPRT5V0U2X:SLPRT5V0U2X
- added R75: 4K, symbol Device:R
- added R76, R77, R78, R79, R80: 10K, symbol Device:R
- added S1, S2: SKHMQLE010, SKHMQLE010:SW_SKHMQLE010, symbol SKHMQLE010:SKHMQLE010
Connections:
- net BOOT: now also C49.2, R75.1, S2.1, S2.2
- net GND: now also C50.1, C51.1, C52.2, Card1.10, Card1.11, Card1.12, Card1.13, Card1.6 (VSS), D8.1, S1.3, S1.4, S1.5, S2.3, S2.4, S2.5
- net RESET: now also C50.2, S1.1, S1.2
- net USB_N: now also D8.3
- net USB_P: now also D8.2
- net VBUS: now also D8.4
- new net: Card1.1 (DAT2), R78.2
- new net: Card1.8 (DAT1), R80.2
- new net MCU_3V3: C51.2, C52.1, Card1.4 (VDD), R75.2, R76.1, R77.1, R78.1, R79.1, R80.1
- new net SD_CS: Card1.2 (CD/DAT3), R77.2
- new net SPI_CLK: Card1.5 (CLX)
- new net SPI_MISO: Card1.3 (CMD), R76.2
- new net SPI_MOSI: Card1.7 (DAT0), R79.2
Other:
- note added: "SWITCH"
- note added: "TF_CARD"
- note added: "USB TYPE C"
- moved on the sheet: J5, R48, R49

Commit message: :clown_face: changed HEIRACHIAL to global
Parts:
- removed R50, R51: 10K, symbol Device:R
- removed R52, R53, R54: 0K, symbol Device:R
- removed U8: BC847BDW1T1G, BC847BDW1T1G:SOT65P210X110-6N, symbol BC847BDW1T1G:BC847BDW1T1G
Other:
- note removed: "BC847BDW1T1G"

Commit message: :tada: Added small changes
Connections:
- no-connect marks 0 -> 4
Changed lines of the file:
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@@
 		(color 0 0 0 0)
+	)
+	(no_connect
+		(at 26.67 43.18)
+	)
+	(no_connect
+		(at 26.67 50.8)
+	)
+	(no_connect
+		(at 62.23 43.18)
+	)
+	(no_connect
+		(at 62.23 50.8)
 	)
 	(wire
@@
 		)
 	)
+	(global_label "DPP_N"
+		(shape input)
+		(at 90.17 76.2 0)
+		(fields_autoplaced yes)
+		(effects
+			(font
+				(size 1.27 1.27)
+			)
+			(justify left)
+		)
+		(property "Intersheetrefs" "${INTERSHEET_REFS}"
+			(at 99.2633 76.2 0)
+			(effects
+				(font
+					(size 1.27 1.27)
+				)
+				(justify left)
+				(hide yes)
+			)
+		)
+	)
+	(global_label "DPP_P"
+		(shape input)
+		(at 90.17 69.85 0)
+		(fields_autoplaced yes)
+		(effects
+			(font
+				(size 1.27 1.27)
+			)
+			(justify left)
+		)
+		(property "Intersheetrefs" "${INTERSHEET_REFS}"
+			(at 99.2028 69.85 0)
+			(effects
+				(font
+					(size 1.27 1.27)
+				)
+				(justify left)
+				(hide yes)
+			)
+		)
+	)
 	(global_label "BOOT"
 		(shape input)
@@
 		)
 	)
-	(hierarchical_label "DPP_N"
-		(shape input)
-		(at 90.17 76.2 0)
-		(effects
-			(font
-				(size 1.27 1.27)
-			)
-			(justify left)
-		)
-	)
-	(hierarchical_label "DPP_P"
-		(shape input)
-		(at 90.17 69.85 0)
-		(effects
-			(font
-				(size 1.27 1.27)
-			)
-			(justify left)
-		)
-	)

Commit message: :tada: Run Electrical rule checker All errors corrected
Parts:
- C49, C50, C51: footprint (none) -> Capacitor_SMD:C_01005_0402Metric
- C52: footprint (none) -> Capacitor_SMD:C_0201_0603Metric
- R48, R49, R75, R76, R77, R78, R79, R80: footprint (none) -> Resistor_SMD:R_01005_0402Metric
Connections:
- net GND: now also C49.1
- no-connect marks 4 -> 5
Changed lines of the file:
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@@
 	)
 	(junction
+		(at 184.15 55.88)
+		(diameter 0)
+		(color 0 0 0 0)
+	)
+	(junction
 		(at 90.17 114.3)
 		(diameter 0)
@@
 		(at 62.23 50.8)
 	)
+	(no_connect
+		(at 72.39 142.24)
+	)
 	(wire
 		(pts
@@
 	(wire
 		(pts
+			(xy 184.15 55.88) (xy 184.15 57.15)
+		)
+		(stroke
+			(width 0)
+			(type default)
+		)
+	)
+	(wire
+		(pts
 			(xy 87.63 151.13) (xy 90.17 151.13)
 		)
@@
 	(wire
 		(pts
+			(xy 220.98 53.34) (xy 220.98 55.88)
+		)
+		(stroke
+			(width 0)
+			(type default)
+		)
+	)
+	(wire
+		(pts
 			(xy 241.3 34.29) (xy 241.3 39.37)
 		)
@@
 	(wire
 		(pts
-			(xy 184.15 54.61) (xy 184.15 57.15)
+			(xy 184.15 54.61) (xy 184.15 55.88)
 		)
 		(stroke
@@
 	(wire
 		(pts
+			(xy 184.15 55.88) (xy 220.98 55.88)
+		)
+		(stroke
+			(width 0)
+			(type default)
+		)
+	)
+	(wire
+		(pts
 			(xy 220.98 39.37) (xy 220.98 36.83)
 		)
@@
 			)
 		)
-		(property "Footprint" ""
+		(property "Footprint" "Resistor_SMD:R_01005_0402Metric"
 			(at 68.072 110.49 90)
 			(effects
@@
 			)
 		)
-		(property "Footprint" ""
+		(property "Footprint" "Capacitor_SMD:C_0201_0603Metric"
 			(at 47.9552 167.64 0)
 			(effects
@@
 			)
 		)
-		(property "Footprint" ""
+		(property "Footprint" "Resistor_SMD:R_01005_0402Metric"
 			(at 51.562 110.49 90)
 			(effects
@@
 			)
 		)
-		(property "Footprint" ""
+		(property "Footprint" "Resistor_SMD:R_01005_0402Metric"
 			(at 64.262 110.49 90)
 			(effects
@@
 			)
 		)
-		(property "Footprint" ""
+		(property "Footprint" "Resistor_SMD:R_01005_0402Metric"
 			(at 60.452 110.49 90)
 			(effects
@@
 			)
 		)
-		(property "Footprint" ""
+		(property "Footprint" "Resistor_SMD:R_01005_0402Metric"
 			(at 82.55 68.072 90)
 			(effects
@@
 			)
 		)
-		(property "Footprint" ""
+		(property "Footprint" "Capacitor_SMD:C_01005_0402Metric"
 			(at 38.4048 160.02 0)
 			(effects
@@
 			)
 		)
-		(property "Footprint" ""
+		(property "Footprint" "Capacitor_SMD:C_01005_0402Metric"
 			(at 220.0148 45.72 0)
 			(effects
@@
 			)
 		)
-		(property "Footprint" ""
+		(property "Footprint" "Resistor_SMD:R_01005_0402Metric"
 			(at 61.468 143.51 90)
 			(effects
@@
 			)
 		)
-		(property "Footprint" ""
+		(property "Footprint" "Capacitor_SMD:C_01005_0402Metric"
 			(at 183.1848 46.99 0)
 			(effects
@@
 			)
 		)
-		(property "Footprint" ""
+		(property "Footprint" "Resistor_SMD:R_01005_0402Metric"
 			(at 82.55 74.422 90)
 			(effects
@@
 			)
 		)
-		(property "Footprint" ""
+		(property "Footprint" "Resistor_SMD:R_01005_0402Metric"
 			(at 222.758 26.67 90)
 			(effects
