File: PLC homemade/OUTPUT.kicad_sch (KiCad schematic)
At the start: 14 parts, among them IC2 PCF8574DGVR, J3 M20-7820646, J4 M20-7820646, U7 SN74HCT14DR

Commit message: :rocket: completed BC847BDW1T1G
Connections:
- net 3V3 renamed 3.3V
Other:
- added sheet Sheet06 (Sheet06.kicad_sch)

Commit message: :tada: COMPLETED SHEET5
Parts:
- added J10, J11, J12, J13, J8, J9: 1729131, 1729131:PHOENIX_1729131, symbol 1729131:1729131
- added RELAY1, RELAY2, RELAY3, RELAY4, RELAY5, RELAY6: G2R-1 DC12, G2R-1 DC12:RELAY-TH_G2R-1, symbol G2R-1 DC12:G2R-1DC12
Connections:
- net 12V: now also RELAY1.5, RELAY2.5, RELAY3.5, RELAY4.5, RELAY5.5, RELAY6.5
- net RLY1: now also RELAY1.1
- net RLY2: now also RELAY2.1
- net RLY3: now also RELAY3.1, RELAY4.1
- net RLY5: now also RELAY5.1
- net RLY6: now also RELAY6.1
- new net COM1: J12.1, RELAY1.2
- new net COM2: J13.1, RELAY2.2
- new net COM3: J8.1, RELAY3.2, RELAY4.2
- new net COM4: J9.1
- new net COM5: J10.1, RELAY5.2
- new net COM6: J11.1, RELAY6.2
- new net NC1: J12.3, RELAY1.3
- new net NC2: J13.3, RELAY2.3
- new net NC3: J8.3, RELAY3.3, RELAY4.3
- new net NC4: J9.3
- new net NC5: J10.3, RELAY5.3
- new net NC6: J11.3, RELAY6.3
- new net NO1: J12.2, RELAY1.4
- new net NO2: J13.2, RELAY2.4
- new net NO3: J8.2, RELAY3.4, RELAY4.4
- new net NO4: J9.2
- new net NO5: J10.2, RELAY5.4
- new net NO6: J11.2, RELAY6.4
Other:
- note added: "OUTPUT"
- note added: "RELAY"
- note added: "TERMINAL BLOCK"
- moved on the sheet: C31, C32, C33, J3, J4, R42, R43, R44, R45, R46, R47, U7

Commit message: :clown_face: changed HEIRACHIAL to global
Changed lines of the file:
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@@
 		)
 	)
-	(hierarchical_label "IIC_SCL"
+	(global_label "IIC_SCL"
 		(shape input)
 		(at 38.1 68.58 180)
+		(fields_autoplaced yes)
 		(effects
 			(font
@@
 			(justify right)
 		)
+		(property "Intersheetrefs" "${INTERSHEET_REFS}"
+			(at 28.16 68.58 0)
+			(effects
+				(font
+					(size 1.27 1.27)
+				)
+				(justify right)
+				(hide yes)
+			)
+		)
 	)
-	(hierarchical_label "IIC_SDA"
+	(global_label "IIC_SDA"
 		(shape input)
 		(at 38.1 66.04 180)
+		(fields_autoplaced yes)
 		(effects
 			(font
@@
 			(justify right)
 		)
+		(property "Intersheetrefs" "${INTERSHEET_REFS}"
+			(at 28.0995 66.04 0)
+			(effects
+				(font
+					(size 1.27 1.27)
+				)
+				(justify right)
+				(hide yes)
+			)
+		)
 	)

Commit message: :tada: Added small changes
Parts:
- added SW1, SW2: SW_Push, symbol Switch:SW_Push
Connections:
- net OT2 is gone; now on net OT1: IC2.5 (P1), J3.2, R43.1, U7.3 (2A)
- net OT3 is gone; now on net OT1: IC2.6 (P2), J3.3, R44.1, U7.5 (3A)
- net OT5 is gone; now on net OT4: IC2.9 (P4), J3.5, R46.1, U7.11 (5A)
- net OT6 is gone; now on net OT4: IC2.10 (P5), J3.6, R47.1, U7.13 (6A)
- net GND: now also SW1.2, SW2.2
- net OT1: now also SW1.1
- net OT4: now also SW2.1

Commit message: :tada: Run Electrical rule checker All errors corrected
Parts:
- added U8: ULN2003ADR, ULN2003ADR:SOIC-16_L9.9-W3.9-P1.27-LS6.0-BL, symbol ULN2003ADR:ULN2003ADR
- C30, C31: footprint (none) -> Capacitor_SMD:C_01005_0402Metric
- C32: footprint (none) -> Capacitor_SMD:CP_Elec_10x7.7
- C33: footprint (none) -> Capacitor_SMD:C_0201_0603Metric
- R42, R43, R44, R45, R46, R47: footprint (none) -> Resistor_SMD:R_01005_0402Metric
- SW1, SW2: footprint (none) -> Button_Switch_SMD:SW_SPST_TL3305A
Connections:
- net 12V: now also U8.9 (COM)
- net COM3: no longer RELAY4.2
- net COM4: now also RELAY4.2
- net GND: now also U8.8 (E)
- net NC3: no longer RELAY4.3
- net NC4: now also RELAY4.3
- net NO3: no longer RELAY4.4
- net NO4: now also RELAY4.4
- net OUT1: now also U8.1 (1B)
- net OUT2: now also U8.2 (2B)
- net OUT3: now also U8.3 (3B)
- net OUT4: now also U8.4 (4B)
- net OUT5: now also U8.5 (5B)
- net OUT6: now also U8.6 (6B)
- net RLY1: now also U8.16 (1C)
- net RLY2: now also U8.15 (2C)
- net RLY3: now also U8.14 (3C); no longer RELAY4.1
- net RLY4: now also RELAY4.1, U8.13 (4C)
- net RLY5: now also U8.12 (5C)
- net RLY6: now also U8.11 (6C)
- no-connect marks 3 -> 5
Other:
- moved on the sheet: J3
