File: PLC homemade/Sheet08.kicad_sch (KiCad schematic)
At the start: 17 parts, among them Q1 AO3400A, Q2 AO3400A, U10 DS1307ZN_, Y2 ABS07-32.768KHZ-T

Commit message: :clown_face: changed HEIRACHIAL to global
Changed lines of the file:
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@@
 		)
 	)
-	(hierarchical_label "IIC_SDA"
+	(global_label "IIC_SDA"
 		(shape input)
 		(at 123.19 48.26 0)
+		(fields_autoplaced yes)
 		(effects
 			(font
@@
 			(justify left)
 		)
+		(property "Intersheetrefs" "${INTERSHEET_REFS}"
+			(at 133.1905 48.26 0)
+			(effects
+				(font
+					(size 1.27 1.27)
+				)
+				(justify left)
+				(hide yes)
+			)
+		)
 	)
-	(hierarchical_label "IIC_SCL"
+	(global_label "IIC_SCL"
 		(shape input)
 		(at 181.61 49.53 0)
+		(fields_autoplaced yes)
 		(effects
 			(font
@@
 			(justify left)
 		)
+		(property "Intersheetrefs" "${INTERSHEET_REFS}"
+			(at 191.55 49.53 0)
+			(effects
+				(font
+					(size 1.27 1.27)
+				)
+				(justify left)
+				(hide yes)
+			)
+		)
 	)

Commit message: :tada: Run Electrical rule checker All errors corrected
Parts:
- C37, C38: footprint (none) -> Capacitor_SMD:C_0201_0603Metric
- C39, C40: footprint (none) -> Capacitor_SMD:C_01005_0402Metric
- R59, R60, R61, R62, R63, R64: footprint (none) -> Resistor_SMD:R_01005_0402Metric
- Y2: footprint (none) -> Crystal:Crystal_SMD_5032-2Pin_5.0x3.2mm
Changed lines of the file:
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@@
 			)
 		)
-		(property "Footprint" ""
+		(property "Footprint" "Capacitor_SMD:C_01005_0402Metric"
 			(at 40.9448 82.55 0)
 			(effects
@@
 			)
 		)
-		(property "Footprint" ""
+		(property "Footprint" "Capacitor_SMD:C_0201_0603Metric"
 			(at 157.1752 102.87 0)
 			(effects
@@
 			)
 		)
-		(property "Footprint" ""
+		(property "Footprint" "Resistor_SMD:R_01005_0402Metric"
 			(at 152.654 48.514 90)
 			(effects
@@
 			)
 		)
-		(property "Footprint" ""
+		(property "Footprint" "Capacitor_SMD:C_0201_0603Metric"
 			(at 139.3952 102.87 0)
 			(effects
@@
 			)
 		)
-		(property "Footprint" ""
+		(property "Footprint" "Resistor_SMD:R_01005_0402Metric"
 			(at 94.234 32.004 90)
 			(effects
@@
 			)
 		)
-		(property "Footprint" ""
+		(property "Footprint" "Resistor_SMD:R_01005_0402Metric"
 			(at 94.234 39.624 90)
 			(effects
@@
 			)
 		)
-		(property "Footprint" ""
+		(property "Footprint" "Capacitor_SMD:C_01005_0402Metric"
 			(at 57.4548 82.55 0)
 			(effects
@@
 			)
 		)
-		(property "Footprint" ""
+		(property "Footprint" "Resistor_SMD:R_01005_0402Metric"
 			(at 152.654 40.894 90)
 			(effects
@@
 			)
 		)
-		(property "Footprint" ""
+		(property "Footprint" "Resistor_SMD:R_01005_0402Metric"
 			(at 94.234 47.244 90)
 			(effects
@@
 			)
 		)
-		(property "Footprint" ""
+		(property "Footprint" "Crystal:Crystal_SMD_5032-2Pin_5.0x3.2mm"
 			(at 49.53 92.71 0)
 			(effects
@@
 			)
 		)
-		(property "Footprint" ""
+		(property "Footprint" "Resistor_SMD:R_01005_0402Metric"
 			(at 152.654 33.274 90)
 			(effects

Commit message: :tada: Arranged the editing
Parts:
- BT1: footprint BK-5058:BAT_BK-5058 -> BatteryHolder_Seiko_MS621F
Changed lines of the file:
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@@
 			)
 		)
-		(property "Footprint" "BK-5058:BAT_BK-5058"
+		(property "Footprint" "BatteryHolder_Seiko_MS621F"
 			(at 38.1 38.1 0)
 			(effects
