File: PLC homemade/PLC homemade.kicad_pcb (KiCad board)
At the start: 2 copper layers, 197 parts, among them IC1 PCF8574DGVR, IC2 PCF8574DGVR, J1 M20-7820646, J10 1729131, J11 1729131, J12 1729131, J13 1729131, J14 Conn_01x02, J15 Conn_01x02, J16 Conn_01x04, J17 Conn_01x02, J2 1803316, J3 M20-7820646, J4 M20-7820646, J5 USB4110GFA, J6 1803316, J7 SS-74810-004, J8 1729131, J9 1729131, Q1 AO3400A, Q2 AO3400A, SW1 SW_Push, SW2 SW_Push, U1 XC6220B331MR, U10 DS1307ZN_, U11 GP8403-TC50-EW_C3152007, U15 EL357N-G, U16 EL357N-G, U17 EL357N-G, U18 EL357N-G, U19 EL357N-G, U20 EL357N-G, U3 W5500, U4 LM324ADT, U5 SN74LVC1G125DRL, U6 SN74LVC1G125DRL, U7 SN74HCT14DR, U8 ULN2003ADR, U9 ESP32-S3-WROOM-1U-N16R8, Y1 Crystal, Y2 ABS07-32.768KHZ-T

Commit message: :ambulance:2CH AND ADC
Parts:
- moved R31 380.1 mm to (59.3, 179.5)
- moved R25 379.6 mm to (54.8, 173.0)
- moved R28 379.1 mm to (59.8, 176.2)
- moved J16 377.6 mm to (43.8, 169.5)
- moved R26 373.5 mm to (60.8, 173.8)
- moved R24 373.0 mm to (60.8, 168.5)
- moved C24 372.5 mm to (59.8, 180.5)
- moved C41 372.2 mm to (85.5, 207.9)
- moved C23 371.3 mm to (60.5, 177.2)
- moved U4 370.1 mm to (61.8, 161.5), turned to -90 degrees
- moved C22 370.0 mm to (60.8, 172.5)
- moved C21 369.9 mm to (60.8, 170.5)
- moved D5 366.4 mm to (56.4, 153.4), turned to 90 degrees
- moved C42 362.7 mm to (85.5, 209.2)
- moved C47 360.9 mm to (73.0, 150.2), turned to 90 degrees
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
Commit message: :ambulance:2output and usbc
Parts:
- moved C28 326.8 mm to (114.5, 184.7), turned to -90 degrees
- moved J1 319.4 mm to (119.0, 184.3), turned to 90 degrees
- moved R29 313.2 mm to (102.0, 175.5)
- moved U6 310.1 mm to (111.3, 185.8)
- moved R34 309.2 mm to (102.0, 179.0)
- moved R33 302.2 mm to (109.5, 175.5)
- moved R35 301.0 mm to (109.5, 179.1)
- moved SW1 297.2 mm to (218.0, 248.0)
- moved SW2 285.3 mm to (231.0, 248.0)
- moved C30 283.8 mm to (219.7, 235.0)
- moved R45 280.1 mm to (200.2, 225.7)
- moved R46 280.1 mm to (200.2, 227.3)
- moved R47 280.1 mm to (200.2, 228.9)
- moved R43 277.8 mm to (219.5, 232.7), turned to -90 degrees
- moved R42 274.6 mm to (219.7, 227.5), turned to -90 degrees
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
Commit message: :tada:Completed most placements in groups
Parts:
- BT1: footprint BK-5058:BAT_BK-5058 -> Battery:BatteryHolder_Seiko_MS621F
- R25: footprint Resistor_SMD:R_01005_0402Metric -> Resistor_SMD:R_1206_3216Metric
- moved C35 284.9 mm to (172.8, 68.5), turned to 180 degrees
- moved C34 283.0 mm to (172.8, 69.5), turned to 180 degrees
- moved C36 282.4 mm to (174.5, 65.8), turned to -90 degrees
- moved R57 280.9 mm to (174.0, 71.0), turned to -90 degrees
- moved R56 279.9 mm to (174.8, 68.0), turned to 180 degrees
- moved R55 278.3 mm to (182.0, 87.2), turned to -90 degrees
- moved R58 265.5 mm to (194.5, 87.7), turned to -90 degrees
- moved U9 256.8 mm to (187.5, 75.6)
- moved J6 232.2 mm to (202.9, 63.7), turned to -90 degrees
- moved R80 231.0 mm to (221.5, 32.7), turned to -90 degrees
- moved R79 229.6 mm to (222.5, 32.8), turned to 90 degrees
- moved C52 229.4 mm to (227.5, 26.8), turned to 90 degrees
- moved R76 223.5 mm to (227.0, 32.7), turned to -90 degrees
- moved C51 223.5 mm to (226.5, 26.8), turned to -90 degrees
- moved R77 222.7 mm to (228.5, 32.3), turned to 90 degrees
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
Commit message: :tada: Arranged the editing
Parts:
- moved J12 146.3 mm to (252.1, 52.6)
- moved J13 146.3 mm to (243.9, 54.8)
- moved SW2 146.0 mm to (135.5, 137.5)
- moved J10 146.0 mm to (251.6, 119.1)
- moved J11 146.0 mm to (243.4, 120.8)
- moved J8 146.0 mm to (252.1, 86.1)
- moved J9 146.0 mm to (252.1, 102.6)
- moved RELAY1 146.0 mm to (226.2, 50.8)
- moved RELAY2 146.0 mm to (226.2, 64.8)
- moved RELAY3 146.0 mm to (226.2, 78.7)
- moved RELAY4 146.0 mm to (226.2, 92.7)
- moved RELAY5 146.0 mm to (226.2, 106.7)
- moved RELAY6 146.0 mm to (226.2, 120.7)
- moved SW1 141.7 mm to (123.9, 142.0)
- moved J3 138.4 mm to (144.0, 130.2)
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
Commit message: :ambulance: Changed the 5 footprint error
Parts:
- added D14: SMBJ7.0CA-Q, SMBJ7.0CA-Q:DIONM5436X244N, F.Cu at (150.0, 89.7)
- added D15: SMBJ7.0CA-Q, SMBJ7.0CA-Q:DIONM5436X244N, F.Cu at (152.5, 96.7)
- added IC3: XL1509-5.0E1, DS1307ZN_:SOIC127P600X175-8N, F.Cu at (87.5, 121.5)
- added IC4: MAX13487EESA+T, DS1307ZN_:SOIC127P600X175-8N, F.Cu at (134.5, 94.7)
- moved R65 291.9 mm to (129.2, 94.2)
- moved C26 266.5 mm to (118.0, 97.2)
- moved C27 266.5 mm to (118.1, 96.2)
- moved C25 266.5 mm to (125.0, 96.2)
- moved R27 266.5 mm to (126.7, 96.2)
- moved U5 266.5 mm to (126.7, 98.5)
- moved R68 246.1 mm to (139.5, 96.5), turned to 90 degrees
- moved F2 245.6 mm to (144.0, 90.3), turned to 90 degrees
- moved F1 244.0 mm to (147.5, 96.6), turned to -90 degrees
- moved R67 242.4 mm to (140.7, 92.7)
- moved R66 241.6 mm to (142.0, 94.7)
- moved C23 6.86 mm to (125.2, 84.0)
- moved R26 6.60 mm to (125.3, 81.5)
- moved C22 6.48 mm to (125.3, 80.5)
- moved J2 6.28 mm to (138.0, 103.3)
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Connections:
- BT1 pad 1: Net-(D10-A) -> (no net)
- BT1 pad 2: AGND -> (no net)

Commit message: :art: wiring componets done
Parts:
- moved SW1 25.5 mm to (100.4, 132.0)
- moved J11 17.2 mm to (251.5, 136.0), turned to 90 degrees
- moved J13 17.1 mm to (252.6, 69.5), turned to 90 degrees
- moved R48 15.7 mm to (183.5, 42.3), turned to 90 degrees
- moved R49 15.0 mm to (184.5, 42.3), turned to 90 degrees
- moved J17 13.9 mm to (137.0, 104.0)
- moved C44 11.1 mm to (124.2, 101.5)
- moved C46 11.1 mm to (127.5, 105.3)
- moved D13 11.1 mm to (130.5, 104.5)
- moved D11 11.1 mm to (125.3, 107.9)
- moved R47 10.9 mm to (132.8, 117.5), turned to 180 degrees
- moved C30 10.9 mm to (137.7, 121.0)
- moved R42 10.9 mm to (137.7, 113.5)
- moved R43 10.9 mm to (137.5, 118.7)
- moved R44 10.9 mm to (137.5, 115.7)
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Connections:
- U11 pad 2: II_SDA -> IIC_SDA
Routing:
- net 3.3V: track 0.00 -> 299.1 mm, vias 0 -> 5
- net 12V: track 0.00 -> 275.4 mm, vias 0 -> 2
- net /ETHERNET/Sheet03/Sheet04/OUTPUT/RLY1: track 0.00 -> 192.7 mm
- net /ETHERNET/Sheet03/Sheet04/OUTPUT/RLY2: track 0.00 -> 172.3 mm
- net /ETHERNET/Sheet03/Sheet04/OUTPUT/RLY3: track 0.00 -> 155.4 mm
- net /ETHERNET/Sheet03/Sheet04/OUTPUT/RLY4: track 0.00 -> 135.6 mm, vias 0 -> 2
- net /ETHERNET/Sheet03/Sheet04/OUTPUT/OT1: track 0.00 -> 121.5 mm, vias 0 -> 2
- net /ETHERNET/Sheet03/Sheet04/OUTPUT/RLY5: track 0.00 -> 117.3 mm, vias 0 -> 2
- net /ETHERNET/Sheet03/Sheet04/OUTPUT/RLY6: track 0.00 -> 98.9 mm
- net IIC_SCL: track 0.00 -> 86.4 mm, vias 0 -> 4
- net SPI_MISO: track 0.00 -> 86.3 mm, vias 0 -> 2
- net 3V3NET: track 0.00 -> 81.2 mm
- net VCC: track 0.00 -> 78.8 mm, vias 0 -> 3
- net IIC_SDA: track 0.00 -> 78.3 mm, vias 0 -> 3
- net SPI_CLK: track 0.00 -> 77.5 mm, vias 0 -> 2
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